Commit message: self collisions enabled

File: signature_ws/src/fyp/urdf/signaturebot_effort_full.urdf (robot description, URDF)
Before this commit: robot signaturebot, 5 links, 4 joints
Joints:
- joint extension: limit lower=0 upper=0.065 effort=100 velocity=0.5 -> lower=0 upper=1 effort=100 velocity=0.5
- joint pitch: limit lower=-1.571 upper=0.698 effort=100 velocity=1.0 -> lower=-3.14 upper=3.14 effort=100 velocity=1.0
- joint yaw: limit lower=-0.96 upper=1.571 effort=100 velocity=1.0 -> lower=-3.14 upper=3.14 effort=100 velocity=1.0
