Commit message: Pre PID Tuning

File: signature_ws/src/fyp/urdf/signaturebot.urdf (robot description, URDF)
Before this commit: robot signaturebot, 5 links, 4 joints
Joints:
- joint joint_p_1: limit lower=-0.79 upper=0.79 effort=30 velocity=0.3 -> lower=-0.79 upper=0.79 effort=100 velocity=0.3
- joint joint_s_1: limit lower=-0.1 upper=0.1 effort=30 velocity=0.05 -> lower=-0.1 upper=0.1 effort=100 velocity=0.05
- joint joint_y_1: limit lower=-0.79 upper=0.79 effort=30 velocity=0.3 -> lower=-0.79 upper=0.79 effort=100 velocity=0.3

Commit message: Xbox Telemetry Complete

File: signature_ws/src/fyp/urdf/signaturebot.urdf (robot description, URDF)
Before this commit: robot signaturebot, 5 links, 4 joints
Joints:
- joint joint_p_1: limit lower=-0.79 upper=0.79 effort=100 velocity=0.3 -> lower=-1.0 upper=1.0 effort=100 velocity=0.3
- joint joint_s_1: limit lower=-0.1 upper=0.1 effort=100 velocity=0.05 -> lower=0 upper=0.05 effort=100 velocity=0.05
- joint joint_y_1: limit lower=-0.79 upper=0.79 effort=100 velocity=0.3 -> lower=-0.6 upper=0.6 effort=100 velocity=0.3

Commit message: collision geometry added

File: signature_ws/src/fyp/urdf/signaturebot.urdf (robot description, URDF)
Before this commit: robot signaturebot, 5 links, 4 joints
Links:
- removed link link_p_1
- removed link link_s_1
- removed link link_y_1
- added link extension_link, mass 0.14210555185115; visual mesh filename=package://fyp/meshes/link_s_1.STL
- added link pitch_link, mass 0.0528284254587736; visual mesh filename=package://fyp/meshes/link_p_1.STL
- added link yaw_link, mass 0.151826725642152; visual mesh filename=package://fyp/meshes/link_y_1.STL
Joints:
- removed joint joint_p_1
- removed joint joint_s_1
- removed joint joint_y_1
- added joint extension: type prismatic, parent yaw_link, child extension_link, origin xyz=0.16609 4E-05 -0.070079 rpy=0 0 0, axis 1 0 0, limit lower=0 upper=0.05 effort=100 velocity=0.05
- added joint pitch: type revolute, parent base_link, child pitch_link, origin xyz=0 0.016806 0.14525 rpy=0 0 0, axis 0 1 0, limit lower=-1.0 upper=1.0 effort=100 velocity=0.3
- added joint yaw: type revolute, parent pitch_link, child yaw_link, origin xyz=0 0 0.02 rpy=0 0 0, axis 0 0 1, limit lower=-0.6 upper=0.6 effort=100 velocity=0.3

File: signature_ws/src/fyp/urdf/signaturebot_effort.urdf (robot description, URDF)
Before this commit: robot signaturebot, 5 links, 4 joints
Links:
- removed link link_p_1
- removed link link_s_1
- removed link link_y_1
- added link extension_link, mass 0.14210555185115; visual mesh filename=package://fyp/meshes/link_s_1.STL
- added link pitch_link, mass 0.0528284254587736; visual mesh filename=package://fyp/meshes/link_p_1.STL
- added link yaw_link, mass 0.151826725642152; visual mesh filename=package://fyp/meshes/link_y_1.STL
Joints:
- removed joint joint_p_1
- removed joint joint_s_1
- removed joint joint_y_1
- added joint extension: type prismatic, parent yaw_link, child extension_link, origin xyz=0.16609 4E-05 -0.070079 rpy=0 0 0, axis 1 0 0, limit lower=0 upper=0.065 effort=100 velocity=0.5
- added joint pitch: type revolute, parent base_link, child pitch_link, origin xyz=0 0.016806 0.14525 rpy=0 0 0, axis 0 1 0, limit lower=-1.571 upper=0.698 effort=100 velocity=1.0
- added joint yaw: type revolute, parent pitch_link, child yaw_link, origin xyz=0 0 0.02 rpy=0 0 0, axis 0 0 1, limit lower=-0.96 upper=1.571 effort=100 velocity=1.0

File: signature_ws/src/fyp/urdf/signaturebot_full.urdf (robot description, URDF)
Before this commit: robot signaturebot, 5 links, 4 joints
Links:
- removed link link_p_1
- removed link link_s_1
- removed link link_y_1
- added link extension_link, mass 0.081074; collision mesh filename=package://fyp/meshes/collision/extension_link.STL; visual mesh filename=package://fyp/meshes/visual/extension_link.STL
- added link pitch_link, mass 0.052828; collision mesh filename=package://fyp/meshes/collision/pitch_link.STL; visual mesh filename=package://fyp/meshes/visual/pitch_link.STL
- added link yaw_link, mass 0.15684; collision mesh filename=package://fyp/meshes/collision/yaw_link.STL; visual mesh filename=package://fyp/meshes/visual/yaw_link.STL
- link base_link: mass 0.352395733896831 -> 0.3524; geometry collision mesh filename=package://fyp/meshes/collision/base_link.STL; visual mesh filename=package://fyp/meshes/visual/base_link.STL
Joints:
- removed joint joint_p_1
- removed joint joint_s_1
- removed joint joint_y_1
- added joint extension: type prismatic, parent yaw_link, child extension_link, origin xyz=0 -3.6757E-05 -0.050079 rpy=-1.5708 0 -1.5708, axis 0 0 1, limit lower=0 upper=0.065 effort=100 velocity=0.5
- added joint pitch: type revolute, parent base_link, child pitch_link, origin xyz=0.096806 0.060005 0.15025 rpy=1.5708 0 1.5708, axis 0 0 1, limit lower=-1.571 upper=0.698 effort=100 velocity=1.0
- added joint yaw: type revolute, parent pitch_link, child yaw_link, origin xyz=0 0 0 rpy=-1.5708 0 0, axis 0 0 -1, limit lower=-0.96 upper=1.571 effort=100 velocity=1.0

Commit message: trajectory data is nice

File: signature_ws/src/fyp/urdf/signaturebot.urdf (robot description, URDF)
Before this commit: robot signaturebot, 5 links, 4 joints
Links:
- link base_link: mass 0.352395733896831 -> 0.3524; geometry collision mesh filename=package://fyp/meshes/collision/base_link.STL; visual mesh filename=package://fyp/meshes/visual/base_link.STL
- link extension_link: mass 0.14210555185115 -> 0.13248; geometry collision mesh filename=package://fyp/meshes/collision/extension_link.STL; visual mesh filename=package://fyp/meshes/visual/extension_link.STL
- link pitch_link: mass 0.0528284254587736 -> 0.039657; geometry collision mesh filename=package://fyp/meshes/collision/pitch_link.STL; visual mesh filename=package://fyp/meshes/visual/pitch_link.STL
- link yaw_link: mass 0.151826725642152 -> 0.17072; geometry collision mesh filename=package://fyp/meshes/collision/yaw_link.STL; visual mesh filename=package://fyp/meshes/visual/yaw_link.STL
Joints:
- joint extension: axis 1 0 0 -> 0 0 1; limit lower=0 upper=0.05 effort=100 velocity=0.05 -> lower=0 upper=0.096 effort=100 velocity=0.5; origin xyz=0.16609 4E-05 -0.070079 rpy=0 0 0 -> xyz=0 -3.6757E-05 -0.050079 rpy=-1.5708 0 -1.5708
- joint pitch: axis 0 1 0 -> 0 0 1; limit lower=-1.0 upper=1.0 effort=100 velocity=0.3 -> lower=-1.5708 upper=1.5708 effort=100 velocity=1.0; origin xyz=0 0.016806 0.14525 rpy=0 0 0 -> xyz=0.096806 0.060005 0.15025 rpy=1.5708 0 1.5708
- joint yaw: axis 0 0 1 -> 0 0 -1; limit lower=-0.6 upper=0.6 effort=100 velocity=0.3 -> lower=-1.5708 upper=1.5708 effort=100 velocity=1.0; origin xyz=0 0 0.02 rpy=0 0 0 -> xyz=0 0 0 rpy=-1.5708 0 0

File: signature_ws/src/fyp/urdf/signaturebot_effort.urdf (robot description, URDF)
Before this commit: robot signaturebot, 5 links, 4 joints
Links:
- link base_link: mass 0.352395733896831 -> 0.3524; geometry collision mesh filename=package://fyp/meshes/collision/base_link.STL; visual mesh filename=package://fyp/meshes/visual/base_link.STL
- link extension_link: mass 0.14210555185115 -> 0.13248; geometry collision mesh filename=package://fyp/meshes/collision/extension_link.STL; visual mesh filename=package://fyp/meshes/visual/extension_link.STL
- link pitch_link: mass 0.0528284254587736 -> 0.039657; geometry collision mesh filename=package://fyp/meshes/collision/pitch_link.STL; visual mesh filename=package://fyp/meshes/visual/pitch_link.STL
- link yaw_link: mass 0.151826725642152 -> 0.17072; geometry collision mesh filename=package://fyp/meshes/collision/yaw_link.STL; visual mesh filename=package://fyp/meshes/visual/yaw_link.STL
Joints:
- joint extension: axis 1 0 0 -> 0 0 1; limit lower=0 upper=0.065 effort=100 velocity=0.5 -> lower=0 upper=0.096 effort=100 velocity=0.5; origin xyz=0.16609 4E-05 -0.070079 rpy=0 0 0 -> xyz=0 4E-05 -0.050079 rpy=-1.5708 0 -1.5708
- joint pitch: axis 0 1 0 -> 0 0 1; limit lower=-1.571 upper=0.698 effort=100 velocity=1.0 -> lower=-3.14 upper=3.14 effort=100 velocity=1.0; origin xyz=0 0.016806 0.14525 rpy=0 0 0 -> xyz=0.096806 0.060005 0.15025 rpy=1.5708 0 1.5708
- joint yaw: axis 0 0 1 -> 0 0 -1; limit lower=-0.96 upper=1.571 effort=100 velocity=1.0 -> lower=-3.14 upper=3.14 effort=100 velocity=1.0; origin xyz=0 0 0.02 rpy=0 0 0 -> xyz=0 0 0 rpy=-1.5708 0 0
