Commit message: dynamic equations added

File: signature_ws/src/fyp/urdf/signaturebot_effort_collision.urdf (robot description, URDF)
Before this commit: robot signaturebot, 5 links, 4 joints
Links:
- link base_link: geometry collision mesh filename=package://fyp/meshes/collision/base_link.STL; visual mesh filename=package://fyp/meshes/collision/base_link.STL
- link extension_link: geometry collision mesh filename=package://fyp/meshes/collision/extension_link.STL; visual mesh filename=package://fyp/meshes/collision/extension_link.STL
- link pitch_link: geometry collision mesh filename=package://fyp/meshes/collision/pitch_link.STL; visual mesh filename=package://fyp/meshes/collision/pitch_link.STL
- link yaw_link: geometry collision mesh filename=package://fyp/meshes/collision/yaw_link.STL; visual mesh filename=package://fyp/meshes/collision/yaw_link.STL
