Commit message: IK Control

File: signature_ws/src/fyp/urdf/signaturebot_effort.urdf (robot description, URDF)
Before this commit: robot signaturebot, 5 links, 4 joints
Joints:
- joint joint_p_1: limit lower=-1.0 upper=1.0 effort=100 velocity=0.3 -> lower=-1.57 upper=1.57 effort=100 velocity=0.3
- joint joint_s_1: limit lower=0 upper=0.05 effort=100 velocity=0.05 -> lower=0 upper=0.06 effort=100 velocity=0.05
- joint joint_y_1: limit lower=-0.6 upper=0.6 effort=100 velocity=0.3 -> lower=-1.57 upper=1.57 effort=100 velocity=0.3

Commit message: Velocity Control Progress

File: signature_ws/src/fyp/urdf/signaturebot_effort.urdf (robot description, URDF)
Before this commit: robot signaturebot, 5 links, 4 joints
Joints:
- joint joint_p_1: limit lower=-1.57 upper=1.57 effort=100 velocity=0.3 -> lower=-1.57 upper=1.57 effort=100 velocity=1.0
- joint joint_s_1: limit lower=0 upper=0.06 effort=100 velocity=0.05 -> lower=0 upper=0.06 effort=100 velocity=0.5
- joint joint_y_1: limit lower=-1.57 upper=1.57 effort=100 velocity=0.3 -> lower=-1.57 upper=1.57 effort=100 velocity=1.0

Commit message: deep copy bullshit

File: signature_ws/src/fyp/urdf/signaturebot_effort.urdf (robot description, URDF)
Before this commit: robot signaturebot, 5 links, 4 joints
Links:
- link extension_link: geometry visual mesh filename=package://fyp/meshes/visual/extension_link.STL
- link pitch_link: geometry visual mesh filename=package://fyp/meshes/visual/pitch_link.STL
- link yaw_link: geometry visual mesh filename=package://fyp/meshes/visual/yaw_link.STL

Commit message: final export & constraint

File: signature_ws/src/fyp/urdf/signaturebot_effort.urdf (robot description, URDF)
Before this commit: robot signaturebot, 5 links, 4 joints
Links:
- link base_link: mass 0.3524 -> 0.35291
- link pitch_link: mass 0.039657 -> 0.034759
- link yaw_link: mass 0.17072 -> 0.17499
Joints:
- joint extension: origin xyz=0 4E-05 -0.050079 rpy=-1.5708 0 -1.5708 -> xyz=0 -0.13608 0 rpy=1.5708 0 0
- joint pitch: origin xyz=0.096806 0.060005 0.15025 rpy=1.5708 0 1.5708 -> xyz=0.09680587 0.060004555 0.15025 rpy=-1.5708 0 1.5708
- joint yaw: origin xyz=0 0 0 rpy=-1.5708 0 0 -> xyz=0 0.050079 3.999E-05 rpy=1.5708 -1.5708 0

File: signature_ws/src/fyp/urdf/signaturebot_effort_collision.urdf (robot description, URDF)
Before this commit: robot signaturebot, 5 links, 4 joints
Links:
- link base_link: mass 0.3524 -> 0.35291
- link pitch_link: mass 0.039657 -> 0.034759
- link yaw_link: mass 0.17072 -> 0.17499
Joints:
- joint extension: origin xyz=0 4E-05 -0.050079 rpy=-1.5708 0 -1.5708 -> xyz=0 -0.13608 0 rpy=1.5708 0 0
- joint pitch: origin xyz=0.096806 0.060005 0.15025 rpy=1.5708 0 1.5708 -> xyz=0.09680587 0.060004555 0.15025 rpy=-1.5708 0 1.5708
- joint yaw: origin xyz=0 0 0 rpy=-1.5708 0 0 -> xyz=0 0.050079 3.999E-05 rpy=1.5708 -1.5708 0

Commit message: i love marco

File: signature_ws/src/fyp/urdf/signaturebot_effort.urdf (robot description, URDF)
Before this commit: robot signaturebot, 5 links, 4 joints
Links:
- link extension_link: geometry collision mesh filename=package://fyp/meshes/collision/extension_link.STL; visual mesh filename=package://fyp/meshes/visual/extension_link.STL
- link pitch_link: geometry collision mesh filename=package://fyp/meshes/collision/pitch_link.STL; visual mesh filename=package://fyp/meshes/visual/pitch_link.STL
- link yaw_link: geometry collision mesh filename=package://fyp/meshes/collision/yaw_link.STL; visual mesh filename=package://fyp/meshes/visual/yaw_link.STL
Joints:
- joint extension: limit lower=0 upper=0.096 effort=100 velocity=0.5 -> lower=-0.005 upper=0.096 effort=100 velocity=0.5
- joint pitch: limit lower=-3.14 upper=3.14 effort=100 velocity=1.0 -> lower=-1.5708 upper=0.8 effort=100 velocity=1.0
- joint yaw: axis 0 0 -1 -> 0 0 1; limit lower=-3.14 upper=3.14 effort=100 velocity=1.0 -> lower=-1.3 upper=1.3 effort=100 velocity=1.0; origin xyz=0 0.050079 3.999E-05 rpy=1.5708 -1.5708 0 -> xyz=0 0.05008 0 rpy=1.5708 -1.5708 0

Commit message: encoder-effort stuff

File: signature_ws/src/fyp/urdf/signaturebot_effort.urdf (robot description, URDF)
Before this commit: robot signaturebot, 5 links, 4 joints
Joints:
- joint extension: limit lower=-0.005 upper=0.096 effort=100 velocity=0.5 -> lower=0.0 upper=0.096 effort=100 velocity=0.5
