Commit message: collision actually finished

File: signature_ws/src/collision_geometry/urdf/collision_geometry.urdf (robot description, URDF)
Before this commit: robot collision_geometry, 4 links, 3 joints
Links:
- removed link yaw_link
- added link yaw_pitch, mass 0.013171; collision mesh filename=package://collision_geometry/meshes/yaw_pitch.STL; visual mesh filename=package://collision_geometry/meshes/yaw_pitch.STL
Joints:
- joint extension: origin xyz=0 -0.0016148 -0.050079 rpy=-1.5708 0 -1.5708 -> xyz=0 4E-05 -0.050079 rpy=-1.5708 0 -1.5708; parent yaw_link -> yaw_pitch
- joint yaw: child yaw_link -> yaw_pitch

File: signature_ws/src/fyp/urdf/signaturebot_effort_full.urdf (robot description, URDF)
Before this commit: robot signaturebot, 5 links, 4 joints
Links:
- link extension_link: mass 0.081074 -> 0.13248
- link pitch_link: mass 0.052828 -> 0.039657
- link yaw_link: mass 0.15684 -> 0.17072
Joints:
- joint extension: origin xyz=0 -3.6757E-05 -0.050079 rpy=-1.5708 0 -1.5708 -> xyz=0 4E-05 -0.050079 rpy=-1.5708 0 -1.5708

File: signature_ws/src/fyp/urdf/signaturebot_full.urdf (robot description, URDF)
Before this commit: robot signaturebot, 5 links, 4 joints
Links:
- link extension_link: mass 0.081074 -> 0.13248
- link pitch_link: mass 0.052828 -> 0.039657
- link yaw_link: mass 0.15684 -> 0.17072
